File: HW/pcb/motiondetector.sch (EAGLE design)
At the start: 15 parts, among them U1 LT1078CN8PBF

Commit message: base PIC24F circuit added
Parts:
- added C6, C8, C9: 100nF, parts:C-EU025-025X050
- added C7: 10uF, parts:CPOL-EUE2.5-5
- added IC1: PIC24FJ32GB002, PIC24FJXXGB0XX :PIC24FJ32GB002
- added R10: 100R, parts:R-EU_0207/10
- added R9: 10k, parts:R-EU_0207/10
- added SV1: (no value), con-lsta:FE05-1
Connections:
- net N$5 renamed ROUT
- new net MCLR: C9.2, R10.2, R9.2, SV1.1
- new net N$12: C7.+, IC1.VCAP/VDDCORE
- new net N$13: IC1.!MCLR, R10.1
- new net PGEC1: IC1.RB1, SV1.5
- new net PGED1: IC1.RB0, SV1.4
- net +3V3: now also C6.2, C8.1, IC1.VDD@1, IC1.VDD@2, R9.1, SV1.2
- net GND: now also C6.1, C7.-, C8.2, C9.1, IC1.DISVREG, IC1.VSS@1, IC1.VSS@2, SV1.3
Other:
- note added: "Debug Header"
- note added: "Radar NF Amplifier"
- moved on the sheet: C1, C2, C3, C4, C5, R1, R2, R3, R4, R5, R6, R7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
